Commit message: update

File: src/reeman_clone_description/urdf/reeman_clone.solidwork.urdf (robot description, URDF)
Before this commit: robot reemen-clone, 7 links, 6 joints
Links:
- added link base_footprint
- added link camera_link
- added link imu_link
- added link lidar_link
- added link three_d_camera_link
- link back_left_caster_link: geometry collision mesh filename=package://reeman_clone_description/meshes/back_left_caster_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; visual mesh filename=package://reeman_clone_description/meshes/back_left_caster_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
- link back_right_caster_link: geometry collision mesh filename=package://reeman_clone_description/meshes/back_right_caster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; visual mesh filename=package://reeman_clone_description/meshes/back_right_caster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
- link base_link: geometry collision mesh filename=package://reeman_clone_description/meshes/base_link.STL; visual mesh filename=package://reeman_clone_description/meshes/base_link.STL
- link front_left_caster_link: geometry collision mesh filename=package://reeman_clone_description/meshes/front_left_caster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; visual mesh filename=package://reeman_clone_description/meshes/front_left_caster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
- link front_right_caster_link: geometry collision mesh filename=package://reeman_clone_description/meshes/front_right_caste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; visual mesh filename=package://reeman_clone_description/meshes/front_right_caste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
- link left_wheel_link: geometry collision mesh filename=package://reeman_clone_description/meshes/left_wheel_link.S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; visual mesh filename=package://reeman_clone_description/meshes/left_wheel_link.S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
- link right_wheel_link: geometry collision mesh filename=package://reeman_clone_description/meshes/right_wheel_link.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; visual mesh filename=package://reeman_clone_description/meshes/right_wheel_link.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
Joints:
- added joint base_footprint_to_base_link: type fixed, parent base_footprint, child base_link, origin xyz=0 0 0 rpy=0 0 0, axis 0 0 0
- added joint camera_link_to_base_link: type fixed, parent base_link, child camera_link, origin xyz=0.1 0 0.1 rpy=0 0 0, axis 0 0 0
- added joint imu_link_to_base_link: type fixed, parent base_link, child imu_link, origin xyz=0.1 0 0.1 rpy=0 0 0, axis 0 0 0
- added joint lidar_link_to_base_link: type fixed, parent base_link, child lidar_link, origin xyz=0.1 0 0.1 rpy=0 0 0, axis 0 0 0
- added joint three_d_camera_link_to_base_link: type fixed, parent base_link, child three_d_camera_link, origin xyz=0.1 0 0.1 rpy=0 0 0, axis 0 0 0
