Commit message: update

File: src/reeman_clone_description/urdf/reeman_clone.solidwork.fortress.urdf.xacro (robot description, xacro)
@@ -3,5 +3,5 @@
      Commit Version: 1.6.0-4-g7f85cfe  Build Version: 1.6.7995.38578
      For more information, please see http://wiki.ros.org/sw_urdf_exporter -->
-<robot name="reeman_clone">
+<robot name="robot">
   <!-- ROM DYNAMICS ADD -->
   <link name="base_footprint"/>
@@ -26,9 +26,9 @@
     <axis xyz="0 0 0"/>
   </joint>
-  <link name="lidar_link"/>
-  <joint name="lidar_link_to_base_link" type="fixed">
+  <link name="laser"/>
+  <joint name="laser_to_base_link" type="fixed">
     <origin xyz="0.1 0 0.1" rpy="0 0 0"/>
     <parent link="base_link"/>
-    <child link="lidar_link"/>
+    <child link="laser"/>
     <axis xyz="0 0 0"/>
   </joint>
@@ -514,5 +514,8 @@
   </gazebo>
   <gazebo>
+    <!-- HARMONIC -->
     <plugin filename="gz_ros2_control-system" name="gz_ros2_control::GazeboSimROS2ControlPlugin">
+    <!-- FORTRESS -->
+    <!-- <plugin filename="ign_ros2_control-system" name="ign_ros2_control::IgnitionROS2ControlSystem"> -->
       <parameters>$(find reeman_clone_description)/config/diff_drive_controller.yaml</parameters>
     </plugin>
@@ -530,5 +533,5 @@
       <update_rate>100</update_rate>
       <visualize>true</visualize>
-      <topic>/usb_imu/data</topic>
+      <topic>imu/out</topic>
       <imu>
         <angular_velocity>
@@ -550,5 +553,5 @@
       <update_rate>100</update_rate>
       <visualize>true</visualize>
-      <topic>/board_imu/data</topic>
+      <topic>imu/wit/out</topic>
       <imu>
         <angular_velocity>
@@ -624,5 +627,5 @@
   </gazebo>
   <!-- GPU Lidar sensor (360° 2D scan) -->
-  <gazebo reference="lidar_link">
+  <gazebo reference="laser">
     <sensor name="gpu_lidar_sensor" type="gpu_lidar">
       <topic>/lidar/scan</topic>

File: src/reeman_clone_description/urdf/reeman_clone.solidwork.urdf (robot description, URDF)
Before this commit: robot reeman_clone, 12 links, 11 joints
Links:
- removed link lidar_link
- added link laser
Joints:
- removed joint lidar_link_to_base_link
- added joint laser_to_base_link: type fixed, parent base_link, child laser, origin xyz=0.1 0 0.1 rpy=0 0 0, axis 0 0 0
