Commit message: update

File: src/reeman_clone_description/urdf/reeman_clone.urdf (robot description, URDF)
Before this commit: robot robot, 12 links, 11 joints
Links:
- removed link base_footprint
- removed link camera_link
- removed link imu_link
- removed link laser
- removed link three_d_camera_link
Joints:
- removed joint base_footprint_to_base_link
- removed joint camera_link_to_base_link
- removed joint imu_link_to_base_link
- removed joint laser_to_base_link
- removed joint three_d_camera_link_to_base_link
