Commit message: update

File: src/reeman_clone_description/urdf/reeman_clone_fortress.urdf.xacro (robot description, xacro)
@@ -2,5 +2,6 @@
 <!-- Derived from `urdf/reemen-clone.urdf` (SolidWorks exporter output). -->
 <robot xmlns:xacro="http://www.ros.org/wiki/xacro" name="reemen">
-  <!-- Mesh paths use `model://my_robot/...` so Gazebo can resolve them via `GZ_SIM_RESOURCE_PATH` / `IGN_GAZEBO_RESOURCE_PATH`. -->
+  <!-- Mesh paths use `package://my_robot/...` so Gazebo can resolve them via `GZ_SIM_RESOURCE_PATH` / `IGN_GAZEBO_RESOURCE_PATH`. -->
+  <xacro:arg name="robot_namespace" default="/"/>
   <link name="base_footprint"/>
   <joint name="base_footprint_joint" type="fixed">
@@ -12,5 +13,5 @@
   <link name="camera_link"/>
   <joint name="camera_link_to_base_link" type="fixed">
-    <origin xyz="0.1 0 0.1" rpy="0 0 0"/>
+    <origin xyz="0.1 0 1.3" rpy="0 0 0"/>
     <parent link="base_link"/>
     <child link="camera_link"/>
@@ -19,5 +20,5 @@
   <link name="three_d_camera_link"/>
   <joint name="three_d_camera_link_to_base_link" type="fixed">
-    <origin xyz="0.1 0 0.1" rpy="0 0 0"/>
+    <origin xyz="0.25 0 0.15" rpy="0 -0.78 0"/>
     <parent link="base_link"/>
     <child link="three_d_camera_link"/>
@@ -26,5 +27,5 @@
   <link name="laser"/>
   <joint name="laser_to_base_link" type="fixed">
-    <origin xyz="0.1 0 0.1" rpy="0 0 0"/>
+    <origin xyz="0.23 0 0.23" rpy="3.14 0 0"/>
     <parent link="base_link"/>
     <child link="laser"/>
@@ -33,5 +34,5 @@
   <link name="usb_imu_link"/>
   <joint name="usb_imu_link_to_base_link" type="fixed">
-    <origin xyz="0.1 0 0.1" rpy="0 0 0"/>
+    <origin xyz="0.07 0 0.05" rpy="0 3.14 -1.57"/>
     <parent link="base_link"/>
     <child link="usb_imu_link"/>
@@ -40,5 +41,5 @@
   <link name="board_imu_link"/>
   <joint name="board_imu_link_to_base_link" type="fixed">
-    <origin xyz="0.1 0 0.1" rpy="0 0 0"/>
+    <origin xyz="0.07 0 0.18" rpy="0 0 3.14"/>
     <parent link="base_link"/>
     <child link="board_imu_link"/>
@@ -68,5 +69,5 @@
       <geometry>
         <mesh
-          filename="model://reeman_clone_description/meshes/base_link.STL" />
+          filename="package://reeman_clone_description/meshes/base_link.STL" />
       </geometry>
       <material
@@ -82,5 +83,5 @@
       <geometry>
         <mesh
-          filename="model://reeman_clone_description/meshes/base_link.STL" />
+          filename="package://reeman_clone_description/meshes/base_link.STL" />
       </geometry>
     </collision>
@@ -108,5 +109,5 @@
       <geometry>
         <mesh
-          filename="model://reeman_clone_description/meshes/right_wheel_link.STL" />
+          filename="package://reeman_clone_description/meshes/right_wheel_link.STL" />
       </geometry>
       <material
@@ -122,5 +123,5 @@
       <geometry>
         <mesh
-          filename="model://reeman_clone_description/meshes/right_wheel_link.STL" />
+          filename="package://reeman_clone_description/meshes/right_wheel_link.STL" />
       </geometry>
     </collision>
@@ -165,5 +166,5 @@
       <geometry>
         <mesh
-          filename="model://reeman_clone_description/meshes/left_wheel_link.STL" />
+          filename="package://reeman_clone_description/meshes/left_wheel_link.STL" />
       </geometry>
       <material
@@ -179,5 +180,5 @@
       <geometry>
         <mesh
-          filename="model://reeman_clone_description/meshes/left_wheel_link.STL" />
+          filename="package://reeman_clone_description/meshes/left_wheel_link.STL" />
       </geometry>
     </collision>
@@ -220,5 +221,5 @@
       <geometry>
         <mesh
-          filename="model://reeman_clone_description/meshes/front_right_caster_link.STL" />
+          filename="package://reeman_clone_description/meshes/front_right_caster_link.STL" />
       </geometry>
       <material
@@ -234,5 +235,5 @@
       <geometry>
         <mesh
-          filename="model://reeman_clone_description/meshes/front_right_caster_link.STL" />
+          filename="package://reeman_clone_description/meshes/front_right_caster_link.STL" />
       </geometry>
     </collision>
@@ -273,5 +274,5 @@
       <geometry>
         <mesh
-          filename="model://reeman_clone_description/meshes/front_left_caster_link.STL" />
+          filename="package://reeman_clone_description/meshes/front_left_caster_link.STL" />
       </geometry>
       <material
@@ -287,5 +288,5 @@
       <geometry>
         <mesh
-          filename="model://reeman_clone_description/meshes/front_left_caster_link.STL" />
+          filename="package://reeman_clone_description/meshes/front_left_caster_link.STL" />
       </geometry>
     </collision>
@@ -326,5 +327,5 @@
       <geometry>
         <mesh
-          filename="model://reeman_clone_description/meshes/back_right_caster_link.STL" />
+          filename="package://reeman_clone_description/meshes/back_right_caster_link.STL" />
       </geometry>
       <material
@@ -340,5 +341,5 @@
       <geometry>
         <mesh
-          filename="model://reeman_clone_description/meshes/back_right_caster_link.STL" />
+          filename="package://reeman_clone_description/meshes/back_right_caster_link.STL" />
       </geometry>
     </collision>
@@ -380,5 +381,5 @@
       <geometry>
         <mesh
-          filename="model://reeman_clone_description/meshes/back_left_caster_link.STL" />
+          filename="package://reeman_clone_description/meshes/back_left_caster_link.STL" />
       </geometry>
       <material
@@ -394,5 +395,5 @@
       <geometry>
         <mesh
-          filename="model://reeman_clone_description/meshes/back_left_caster_link.STL" />
+          filename="package://reeman_clone_description/meshes/back_left_caster_link.STL" />
       </geometry>
     </collision>
@@ -519,47 +520,81 @@
   </gazebo>
   <!-- IMU sensors -->
-  <gazebo reference="usb_imu_link">
-    <sensor name="usb_imu_sensor" type="imu">
+<gazebo reference="usb_imu_link">
+  <sensor name="usb_imu_sensor" type="imu">
+    <always_on>1</always_on>
+    <update_rate>100</update_rate>
+    <visualize>true</visualize>
+    <topic>/imu/out</topic>
+    <gz_frame_id>usb_imu_link</gz_frame_id>
+    <imu>
+      <angular_velocity>
+        <x><noise type="gaussian"><mean>0.0</mean><stddev>2e-4</stddev></noise></x>
+        <y><noise type="gaussian"><mean>0.0</mean><stddev>2e-4</stddev></noise></y>
+        <z><noise type="gaussian"><mean>0.0</mean><stddev>2e-4</stddev></noise></z>
+      </angular_velocity>
+      <linear_acceleration>
+        <x><noise type="gaussian"><mean>0.0</mean><stddev>1.7e-2</stddev></noise></x>
+        <y><noise type="gaussian"><mean>0.0</mean><stddev>1.7e-2</stddev></noise></y>
+        <z><noise type="gaussian"><mean>0.0</mean><stddev>1.7e-2</stddev></noise></z>
+      </linear_acceleration>
+    </imu>
+  </sensor>
+</gazebo>
+<gazebo reference="board_imu_link">
+  <sensor name="board_imu_sensor" type="imu">
+    <always_on>1</always_on>
+    <update_rate>100</update_rate>
+    <visualize>true</visualize>
+    <topic>/imu/wit/out</topic>
+    <gz_frame_id>board_imu_link</gz_frame_id>
+    <imu>
+      <angular_velocity>
+        <x><noise type="gaussian"><mean>0.0</mean><stddev>2e-4</stddev></noise></x>
+        <y><noise type="gaussian"><mean>0.0</mean><stddev>2e-4</stddev></noise></y>
+        <z><noise type="gaussian"><mean>0.0</mean><stddev>2e-4</stddev></noise></z>
+      </angular_velocity>
+      <linear_acceleration>
+        <x><noise type="gaussian"><mean>0.0</mean><stddev>1.7e-2</stddev></noise></x>
+        <y><noise type="gaussian"><mean>0.0</mean><stddev>1.7e-2</stddev></noise></y>
+        <z><noise type="gaussian"><mean>0.0</mean><stddev>1.7e-2</stddev></noise></z>
+      </linear_acceleration>
+    </imu>
+  </sensor>
+</gazebo>
+  <!-- RGB Camera sensor -->
+<gazebo reference="camera_link">
+  <sensor name="camera_sensor" type="camera">
+    <ign_frame_id>camera_link_optical</ign_frame_id>
+    <update_rate>30</update_rate>
+    <always_on>1</always_on>
+    <visualize>true</visualize>
+    <topic>/camera/image_raw</topic>
+    <camera>
+      <horizontal_fov>1.047</horizontal_fov>
+      <image>
+        <width>640</width>
+        <height>480</height>
+        <format>R8G8B8</format>
+      </image>
+      <clip>
+        <near>0.1</near>
+        <far>100.0</far>
+      </clip>
+      <noise>
+        <type>gaussian</type>
+        <mean>0.0</mean>
+        <stddev>0.007</stddev>
+      </noise>
+    </camera>
+  </sensor>
+</gazebo>
+  <!-- 3D Camera (RGBD) sensor -->
+  <gazebo reference="three_d_camera_link">
+    <sensor name="rgbd_camera_sensor" type="rgbd_camera">
+      <update_rate>30</update_rate>
       <always_on>1</always_on>
-      <update_rate>100</update_rate>
       <visualize>true</visualize>
-      <topic>imu/out</topic>
-      <imu>
-        <angular_velocity>
-          <x><noise type="gaussian"><mean>0</mean><stddev>2e-4</stddev></noise></x>
-          <y><noise type="gaussian"><mean>0</mean><stddev>2e-4</stddev></noise></y>
-          <z><noise type="gaussian"><mean>0</mean><stddev>2e-4</stddev></noise></z>
-        </angular_velocity>
-        <linear_acceleration>
-          <x><noise type="gaussian"><mean>0</mean><stddev>1.7e-2</stddev></noise></x>
-          <y><noise type="gaussian"><mean>0</mean><stddev>1.7e-2</stddev></noise></y>
-          <z><noise type="gaussian"><mean>0</mean><stddev>1.7e-2</stddev></noise></z>
-        </linear_acceleration>
-      </imu>
-    </sensor>
-  </gazebo>
-  <gazebo reference="board_imu_link">
-    <sensor name="board_imu_sensor" type="imu">
-      <always_on>1</always_on>
-      <update_rate>100</update_rate>
-      <visualize>true</visualize>
-      <topic>imu/wit/out</topic>
-      <imu>
-        <angular_velocity>
-          <x><noise type="gaussian"><mean>0</mean><stddev>2e-4</stddev></noise></x>
-          <y><noise type="gaussian"><mean>0</mean><stddev>2e-4</stddev></noise></y>
-          <z><noise type="gaussian"><mean>0</mean><stddev>2e-4</stddev></noise></z>
-        </angular_velocity>
-        <linear_acceleration>
-          <x><noise type="gaussian"><mean>0</mean><stddev>1.7e-2</stddev></noise></x>
-          <y><noise type="gaussian"><mean>0</mean><stddev>1.7e-2</stddev></noise></y>
-          <z><noise type="gaussian"><mean>0</mean><stddev>1.7e-2</stddev></noise></z>
-        </linear_acceleration>
-      </imu>
-    </sensor>
-  </gazebo>
-  <!-- RGB Camera sensor -->
-  <gazebo reference="camera_link">
-    <sensor name="camera_sensor" type="camera">
+      <topic>/three_d_camera</topic>
+      <gz_frame_id>three_d_camera_link_optical</gz_frame_id>
       <camera>
         <horizontal_fov>1.047</horizontal_fov>
@@ -571,35 +606,8 @@
         <clip>
           <near>0.1</near>
-          <far>100</far>
-        </clip>
+          <far>10.0</far> </clip>
         <noise>
           <type>gaussian</type>
-          <mean>0</mean>
-          <stddev>0.007</stddev>
-        </noise>
-      </camera>
-      <always_on>1</always_on>
-      <update_rate>30</update_rate>
-      <visualize>true</visualize>
-      <topic>/camera/image_raw</topic>
-    </sensor>
-  </gazebo>
-  <!-- 3D Camera (RGBD) sensor -->
-  <gazebo reference="three_d_camera_link">
-    <sensor name="rgbd_camera_sensor" type="rgbd_camera">
-      <camera>
-        <horizontal_fov>1.047</horizontal_fov>
-        <image>
-          <width>640</width>
-          <height>480</height>
-          <format>R8G8B8</format>
-        </image>
-        <clip>
-          <near>0.1</near>
-          <far>10</far>
-        </clip>
-        <noise>
-          <type>gaussian</type>
-          <mean>0</mean>
+          <mean>0.0</mean>
           <stddev>0.007</stddev>
         </noise>
@@ -607,12 +615,8 @@
           <clip>
             <near>0.1</near>
-            <far>10</far>
+            <far>10.0</far>
           </clip>
         </depth_camera>
       </camera>
-      <always_on>1</always_on>
-      <update_rate>30</update_rate>
-      <visualize>true</visualize>
-      <topic>/three_d_camera</topic>
     </sensor>
   </gazebo>
@@ -621,6 +625,7 @@
     <sensor name="gpu_lidar_sensor" type="gpu_lidar">
       <topic>/lidar/scan</topic>
+      <gz_frame_id>laser</gz_frame_id>
       <update_rate>10</update_rate>
-      <ray>
+      <lidar>
         <scan>
           <horizontal>
@@ -647,5 +652,5 @@
           <stddev>0.01</stddev>
         </noise>
-      </ray>
+      </lidar>
       <always_on>1</always_on>
       <visualize>true</visualize>
@@ -654,4 +659,7 @@
   <gazebo>
     <plugin filename="gz_ros2_control-system" name="gz_ros2_control::GazeboSimROS2ControlPlugin">
+      <!-- <ros>
+        <namespace>"default_robot1"</namespace>
+      </ros> -->
       <parameters>$(find reeman_clone_description)/config/diff_drive_controller.yaml</parameters>
     </plugin>

Commit message: update

File: src/reeman_clone_description/urdf/reeman_clone_fortress.urdf.xacro (robot description, xacro)
@@ -73,6 +73,6 @@
       <material
         name="">
-        <color
-          rgba="0.62745 0.62745 0.62745 1" />
+        <!-- <color rgba="0.62745 0.62745 0.62745 1" /> -->
+        <color rgba="1.0 0.5 0.0 1.0" />
       </material>
     </visual>
@@ -427,4 +427,14 @@
     </joint>
   </ros2_control>
+  <!-- COLOR -->
+  <gazebo reference="base_link">
+    <material>Gazebo/Orange</material>
+  </gazebo>
+  <gazebo reference="left_wheel_link">
+    <material>Gazebo/Black</material>
+  </gazebo>
+  <gazebo reference="right_wheel_link">
+    <material>Gazebo/Black</material>
+  </gazebo>
   <!-- === Wheel friction: HIGH so wheels grip the ground and propel the robot === -->
   <gazebo reference="left_wheel_link">

Commit message: psa

File: src/reeman_clone_description/urdf/reeman_clone_fortress.urdf.xacro (robot description, xacro)
@@ -51,16 +51,12 @@
     name="base_link">
     <inertial>
-      <origin
-        xyz="-0.006381 0.0039481 0.0009"
-        rpy="0 0 0" />
-      <mass
-        value="0.2471" />
-      <inertia
-        ixx="0.0033314"
-        ixy="-3.3441E-08"
-        ixz="-4.1779E-18"
-        iyy="0.0049517"
-        iyz="-2.0567E-19"
-        izz="0.008283" />
+      <origin xyz="-0.02 0.0 -0.05" rpy="0 0 0" />
+      <mass value="10.0" /> <inertia
+        ixx="0.077"
+        ixy="0"
+        ixz="0"
+        iyy="0.108"
+        iyz="0"
+        izz="0.161" />
     </inertial>
     <visual>
@@ -446,8 +442,8 @@
         <contact>
           <ode>
-            <kp>2e5</kp>
-            <kd>20.0</kd>
-            <max_vel>0.03</max_vel>
-            <min_depth>0.0003</min_depth>
+            <kp>1e7</kp>
+            <kd>1.0</kd>
+            <max_vel>0.01</max_vel>
+            <min_depth>0.001</min_depth>
           </ode>
         </contact>
@@ -473,8 +469,8 @@
         <contact>
           <ode>
-            <kp>2e5</kp>
-            <kd>20.0</kd>
-            <max_vel>0.03</max_vel>
-            <min_depth>0.0003</min_depth>
+            <kp>1e7</kp>
+            <kd>1.0</kd>
+            <max_vel>0.01</max_vel>
+            <min_depth>0.001</min_depth>
           </ode>
         </contact>
@@ -489,5 +485,5 @@
           <ode><mu>0.0</mu><mu2>0.0</mu2></ode>
         </friction>
-        <contact><ode><kp>1e5</kp><kd>10</kd></ode></contact>
+	<contact><ode><kp>1e7</kp><kd>1.0</kd><max_vel>0.01</max_vel><min_depth>0.001</min_depth></ode></contact>
       </surface>
     </collision>
@@ -499,5 +495,5 @@
           <ode><mu>0.0</mu><mu2>0.0</mu2></ode>
         </friction>
-        <contact><ode><kp>1e5</kp><kd>10</kd></ode></contact>
+	<contact><ode><kp>1e7</kp><kd>1.0</kd><max_vel>0.01</max_vel><min_depth>0.001</min_depth></ode></contact>
       </surface>
     </collision>
@@ -509,5 +505,5 @@
           <ode><mu>0.0</mu><mu2>0.0</mu2></ode>
         </friction>
-        <contact><ode><kp>1e5</kp><kd>10</kd></ode></contact>
+	<contact><ode><kp>1e7</kp><kd>1.0</kd><max_vel>0.01</max_vel><min_depth>0.001</min_depth></ode></contact>
       </surface>
     </collision>
@@ -519,5 +515,5 @@
           <ode><mu>0.0</mu><mu2>0.0</mu2></ode>
         </friction>
-        <contact><ode><kp>1e5</kp><kd>10</kd></ode></contact>
+	<contact><ode><kp>1e7</kp><kd>1.0</kd><max_vel>0.01</max_vel><min_depth>0.001</min_depth></ode></contact>
       </surface>
     </collision>
